Commit message: Add sim-to-sim terrain heightmap support

File: legged_robot_description/go2_description/urdf/robot.xacro (robot description, xacro)
@@ -5,4 +5,6 @@
     <xacro:arg name="enable_sim" default="true" />
     <xacro:arg name="enable_lowlevel_write" default="true" />
+    <xacro:arg name="lowstate_topic" default="/lowstate" />
+    <xacro:arg name="lowcmd_topic" default="/lowcmd" />
     <xacro:include filename="$(find go2_description)/urdf/const.xacro"/>
     <xacro:include filename="$(find go2_description)/urdf/materials.xacro"/>
@@ -132,4 +134,6 @@
         prefix="$(arg prefix)"
         enable_sim="$(arg enable_sim)"
-        enable_lowlevel_write="$(arg enable_lowlevel_write)"/>
+        enable_lowlevel_write="$(arg enable_lowlevel_write)"
+        lowstate_topic="$(arg lowstate_topic)"
+        lowcmd_topic="$(arg lowcmd_topic)"/>
 </robot>

File: legged_robot_description/go2_description/urdf/ros2_control.xacro (robot description, xacro)
@@ -1,5 +1,5 @@
 <?xml version="1.0"?>
 <robot xmlns:xacro="http://www.ros.org/wiki/xacro">
-  <xacro:macro name="go2_ros2_control" params="prefix enable_sim:=false enable_lowlevel_write:=true">
+  <xacro:macro name="go2_ros2_control" params="prefix enable_sim:=false enable_lowlevel_write:=true lowstate_topic:=/lowstate lowcmd_topic:=/lowcmd">
     <ros2_control name="go2_ros2_control" type="system">
       <!-- This plugin has been deprecated, so enable_sim should always be false -->
@@ -13,4 +13,6 @@
           <plugin>legged_ros2_control/Go2SystemInterface</plugin>
           <param name="enable_lowlevel_write">${enable_lowlevel_write}</param>
+          <param name="lowstate_topic">${lowstate_topic}</param>
+          <param name="lowcmd_topic">${lowcmd_topic}</param>
         </hardware>
       </xacro:unless>
